Commit message: feat(urdf): update robot_description with lumi_small_robot URDF model

File: luminax_ws/src/luminax_description/urdf/luminax.urdf.xacro (robot description, xacro)
@@ -1,61 +1,87 @@
 <?xml version="1.0"?>
 <!-- =====================================================================
-     LUMINAX / LUMI  -  robot description (navigation base, no arm)
+     LUMINAX / LUMI  -  Robot Description (Accurate Physical Model)
      ROS 2 Jazzy
-     TF chain produced by this file (via robot_state_publisher):
-         base_footprint -> base_link -> { laser_frame, camera_link, imu_link,
-                                          body_link, wheels, caster }
-     The odom->base_footprint transform is NOT here; it comes from
-     rf2o_laser_odometry.  map->odom comes from slam_toolbox / AMCL.
-     >>> EVERY NUMBER MARKED  (MEASURE)  MUST BE REPLACED WITH A REAL
-     >>> MEASUREMENT FROM YOUR BUILT ROBOT BEFORE NAVIGATION WILL BE ACCURATE.
+     Modeled with exact measurements from physical robot photos using a
+     15 cm DOMS engineering scale reference.
+     Physical Specifications:
+       - Drive Type: 4WD Skid-Steer (4 x Yellow DC TT Gear Motors)
+       - Wheels: 65mm dia x 26mm width (Yellow rims + Black treaded tires)
+       - Wheel Separation (Track Width): 0.178 m (center-to-center)
+       - Wheelbase (Front-to-Rear Axle): 0.145 m
+       - Lower Deck: 0.190 m x 0.140 m black acrylic chassis
+       - Standoffs: 0.040 m (40 mm) brass hex spacers
+       - Upper Deck: 0.180 m x 0.165 m white acrylic mounting deck
+       - 2D LiDAR: Slamtec RPLiDAR A1 on elevated black mount
+       - LiDAR Optical Scan Plane: z = 0.175 m above floor
+       - Head Enclosure: 3D-printed white companion shell with screen bezel
      ===================================================================== -->
 <robot name="luminax" xmlns:xacro="http://www.ros.org/wiki/xacro">
   <!-- ============================================================
-       TUNABLE PARAMETERS  -  edit these after measuring the robot
-       ============================================================ -->
-  <!-- Drive geometry (CRITICAL for odometry & navigation) -->
-  <xacro:property name="wheel_radius"     value="0.045"/>  <!-- (MEASURE) wheel radius [m]. 90mm dia wheel -> 0.045 -->
-  <xacro:property name="wheel_width"      value="0.035"/>  <!-- (MEASURE) wheel width [m] -->
-  <xacro:property name="wheel_separation" value="0.375"/>  <!-- (MEASURE) distance between the two drive-wheel contact points [m] -->
-  <xacro:property name="wheel_mass"       value="0.20"/>
-  <!-- Chassis base box (the lower deck that carries motors/battery) -->
-  <xacro:property name="base_x"   value="0.40"/>   <!-- (MEASURE) length -->
-  <xacro:property name="base_y"   value="0.34"/>   <!-- (MEASURE) width  -->
-  <xacro:property name="base_z"   value="0.12"/>   <!-- (MEASURE) height of base box -->
-  <xacro:property name="base_mass" value="8.0"/>   <!-- (MEASURE) -->
-  <!-- Height of the wheel axle above the ground.
-       For a wheel of radius r sitting on the floor, the axle is at z = r. -->
-  <xacro:property name="axle_height" value="${wheel_radius}"/>
-  <!-- LiDAR mounting offset RELATIVE TO base_link origin (CRITICAL).
-       base_link origin sits on the ground directly, so these are
-       measured from the point on the floor between the drive wheels. -->
-  <xacro:property name="lidar_x"   value="0.13"/>  <!-- (MEASURE) forward offset of LiDAR centre [m] -->
-  <xacro:property name="lidar_y"   value="0.0"/>   <!-- (MEASURE) left/right offset [m] -->
-  <xacro:property name="lidar_z"   value="0.22"/>  <!-- (MEASURE) height of LiDAR scan plane above ground [m] -->
-  <xacro:property name="lidar_yaw" value="0.0"/>   <!-- (MEASURE) yaw of the LiDAR 0-angle vs robot +X [rad].
-                                                        Many RPLiDAR A1 mounts have the cable/0 pointing BACKWARD;
-                                                        if your /scan looks rotated 180 deg, set this to 3.14159. -->
-  <!-- Camera mounting offset relative to base_link -->
-  <xacro:property name="camera_x" value="0.155"/> <!-- (MEASURE) -->
-  <xacro:property name="camera_y" value="0.0"/>   <!-- (MEASURE) -->
-  <xacro:property name="camera_z" value="0.85"/>  <!-- (MEASURE) height of camera above ground [m] -->
-  <!-- IMU mounting offset relative to base_link (optional sensor) -->
-  <xacro:property name="imu_x" value="0.0"/>
-  <xacro:property name="imu_y" value="0.0"/>
-  <xacro:property name="imu_z" value="0.18"/>
-  <!-- Caster offset relative to base_link -->
-  <xacro:property name="caster_x" value="-0.14"/> <!-- (MEASURE) rear offset -->
-  <xacro:property name="caster_radius" value="0.02"/>
-  <xacro:property name="PI" value="3.14159265359"/>
-  <!-- ============================================================
-       Materials
-       ============================================================ -->
-  <material name="body_white"><color rgba="0.92 0.92 0.92 1.0"/></material>
-  <material name="dark">      <color rgba="0.10 0.10 0.10 1.0"/></material>
-  <material name="sensor_black"><color rgba="0.03 0.03 0.03 1.0"/></material>
-  <material name="accent">    <color rgba="0.55 0.45 0.85 1.0"/></material>
-  <!-- ============================================================
-       Reusable inertia macros
+       CALIBRATED PHYSICAL PARAMETERS (from 15cm DOMS Scale Reference)
+       ============================================================ -->
+  <!-- Drive Geometry -->
+  <xacro:property name="wheel_radius"     value="0.0325"/>  <!-- 65 mm diameter TT wheel -> r = 32.5 mm -->
+  <xacro:property name="wheel_width"      value="0.026"/>   <!-- 26 mm wheel tread width -->
+  <xacro:property name="wheel_separation" value="0.178"/>   <!-- 178 mm track width (150 mm inner distance + 26 mm tire) -->
+  <xacro:property name="wheelbase"        value="0.145"/>   <!-- 145 mm front-to-rear axle distance -->
+  <xacro:property name="wheel_mass"       value="0.045"/>   <!-- ~45 g per wheel -->
+  <!-- Lower Chassis (Black Acrylic Base + Motor Brackets) -->
+  <xacro:property name="lower_deck_x"     value="0.190"/>   <!-- 190 mm length -->
+  <xacro:property name="lower_deck_y"     value="0.140"/>   <!-- 140 mm width -->
+  <xacro:property name="lower_deck_z"     value="0.003"/>   <!-- 3 mm acrylic plate -->
+  <xacro:property name="lower_deck_z_pos" value="0.0765"/>  <!-- Lower plate center sits 76.5 mm above ground -->
+  <xacro:property name="lower_deck_mass"  value="0.95"/>    <!-- Lower chassis, battery pack, motor drivers ~ 0.95 kg -->
+  <!-- Brass Standoffs -->
+  <xacro:property name="standoff_h"       value="0.040"/>   <!-- Exactly 40 mm brass standoffs (verified Page 2) -->
+  <xacro:property name="standoff_r"       value="0.003"/>   <!-- 6 mm diameter -->
+  <!-- Upper Chassis (White Acrylic Deck) -->
+  <xacro:property name="upper_deck_x"     value="0.180"/>   <!-- 180 mm length -->
+  <xacro:property name="upper_deck_y"     value="0.165"/>   <!-- 165 mm width (verified Page 3) -->
+  <xacro:property name="upper_deck_z"     value="0.005"/>   <!-- 5 mm acrylic plate -->
+  <xacro:property name="upper_deck_z_pos" value="0.1205"/>  <!-- Upper plate center sits 120.5 mm above ground -->
+  <xacro:property name="upper_deck_mass"  value="0.35"/>    <!-- Upper deck plate + hardware ~ 0.35 kg -->
+  <!-- LiDAR Sensor (Slamtec RPLiDAR A1) -->
+  <xacro:property name="lidar_riser_x"    value="0.120"/>   <!-- Black riser plate length -->
+  <xacro:property name="lidar_riser_y"    value="0.095"/>   <!-- Black riser plate width -->
+  <xacro:property name="lidar_riser_z"    value="0.003"/>
+  <xacro:property name="lidar_x"          value="0.045"/>   <!-- Mounted forward on upper deck (+45 mm) -->
+  <xacro:property name="lidar_y"          value="0.000"/>   <!-- Centered laterally -->
+  <xacro:property name="lidar_z"          value="0.175"/>   <!-- Exact optical scan plane height = 175 mm above ground (Page 4) -->
+  <xacro:property name="lidar_yaw"        value="0.0"/>     <!-- Default forward heading (set 3.14159 if cable orientation requires) -->
+  <xacro:property name="lidar_mass"       value="0.17"/>    <!-- 170 g RPLiDAR A1 -->
+  <!-- 3D Printed Head / Body Shell -->
+  <xacro:property name="head_x"           value="-0.035"/>  <!-- Mounted rearward to clear LiDAR beam -->
+  <xacro:property name="head_z"           value="0.235"/>   <!-- Center height of body shell -->
+  <xacro:property name="head_length"      value="0.110"/>
+  <xacro:property name="head_width"       value="0.160"/>
+  <xacro:property name="head_height"      value="0.220"/>
+  <xacro:property name="head_mass"        value="0.45"/>    <!-- Shell + Raspberry Pi 5 + display ~ 0.45 kg -->
+  <!-- Camera Offset (inside head screen bezel) -->
+  <xacro:property name="camera_x"         value="0.025"/>
+  <xacro:property name="camera_y"         value="0.000"/>
+  <xacro:property name="camera_z"         value="0.305"/>   <!-- 305 mm above ground -->
+  <!-- IMU Offset (on lower deck) -->
+  <xacro:property name="imu_x"            value="0.000"/>
+  <xacro:property name="imu_y"            value="0.000"/>
+  <xacro:property name="imu_z"            value="0.082"/>
+  <!-- Wheel Axle Height above ground -->
+  <xacro:property name="axle_height"      value="${wheel_radius}"/>
+  <xacro:property name="PI"               value="3.14159265359"/>
+  <!-- ============================================================
+       COLOR MATERIALS
+       ============================================================ -->
+  <material name="chassis_black"><color rgba="0.08 0.08 0.08 1.0"/></material>
+  <material name="deck_white">   <color rgba="0.96 0.96 0.96 1.0"/></material>
+  <material name="shell_white">  <color rgba="0.93 0.93 0.94 1.0"/></material>
+  <material name="rim_yellow">   <color rgba="0.98 0.80 0.08 1.0"/></material>
+  <material name="motor_yellow"> <color rgba="0.95 0.74 0.05 1.0"/></material>
+  <material name="rubber_black"> <color rgba="0.12 0.12 0.12 1.0"/></material>
+  <material name="brass_gold">   <color rgba="0.82 0.68 0.28 1.0"/></material>
+  <material name="sensor_black"> <color rgba="0.03 0.03 0.03 1.0"/></material>
+  <material name="screen_dark">  <color rgba="0.10 0.14 0.20 1.0"/></material>
+  <material name="accent_blue">  <color rgba="0.15 0.50 0.85 1.0"/></material>
+  <!-- ============================================================
+       REUSABLE INERTIA MACROS
        ============================================================ -->
   <xacro:macro name="box_inertia" params="m x y z">
@@ -76,22 +102,91 @@
   </xacro:macro>
   <!-- ============================================================
-       base_footprint : the ground-projected root frame
-       ============================================================ -->
+       1. ROOT FRAMES
+       ============================================================ -->
+  <!-- base_footprint : Ground projection at z = 0 -->
   <link name="base_footprint"/>
-  <!-- ============================================================
-       base_link : main chassis.  Its origin is on the floor,
-       centred between the drive wheels (standard convention).
-       ============================================================ -->
+  <!-- base_link : Main reference frame on the ground plane at robot footprint center -->
   <link name="base_link">
-    <visual>
-      <origin xyz="0 0 ${axle_height + base_z/2}" rpy="0 0 0"/>
-      <geometry><box size="${base_x} ${base_y} ${base_z}"/></geometry>
-      <material name="body_white"/>
-    </visual>
-    <collision>
-      <origin xyz="0 0 ${axle_height + base_z/2}" rpy="0 0 0"/>
-      <geometry><box size="${base_x} ${base_y} ${base_z}"/></geometry>
-    </collision>
-    <xacro:box_inertia m="${base_mass}" x="${base_x}" y="${base_y}" z="${base_z}"/>
+    <!-- Visual: Lower Chassis Black Plate -->
+    <visual>
+      <origin xyz="0 0 ${lower_deck_z_pos}" rpy="0 0 0"/>
+      <geometry><box size="${lower_deck_x} ${lower_deck_y} ${lower_deck_z}"/></geometry>
+      <material name="chassis_black"/>
+    </visual>
+    <collision>
+      <origin xyz="0 0 ${lower_deck_z_pos}" rpy="0 0 0"/>
+      <geometry><box size="${lower_deck_x} ${lower_deck_y} ${lower_deck_z}"/></geometry>
+    </collision>
+    <!-- Visual: Left Bracket Leg -->
+    <visual>
+      <origin xyz="0 0.060 ${(lower_deck_z_pos + axle_height)/2}" rpy="0 0 0"/>
+      <geometry><box size="0.160 0.012 ${lower_deck_z_pos - axle_height + 0.01}"/></geometry>
+      <material name="chassis_black"/>
+    </visual>
+    <!-- Visual: Right Bracket Leg -->
+    <visual>
+      <origin xyz="0 -0.060 ${(lower_deck_z_pos + axle_height)/2}" rpy="0 0 0"/>
+      <geometry><box size="0.160 0.012 ${lower_deck_z_pos - axle_height + 0.01}"/></geometry>
+      <material name="chassis_black"/>
+    </visual>
+    <!-- Visual: 4 Yellow TT Gear Motor Bodies -->
+    <visual>
+      <origin xyz="${wheelbase/2} 0.062 ${axle_height}" rpy="0 0 0"/>
+      <geometry><box size="0.065 0.022 0.020"/></geometry>
+      <material name="motor_yellow"/>
+    </visual>
+    <visual>
+      <origin xyz="${wheelbase/2} -0.062 ${axle_height}" rpy="0 0 0"/>
+      <geometry><box size="0.065 0.022 0.020"/></geometry>
+      <material name="motor_yellow"/>
+    </visual>
+    <visual>
+      <origin xyz="${-wheelbase/2} 0.062 ${axle_height}" rpy="0 0 0"/>
+      <geometry><box size="0.065 0.022 0.020"/></geometry>
+      <material name="motor_yellow"/>
+    </visual>
+    <visual>
+      <origin xyz="${-wheelbase/2} -0.062 ${axle_height}" rpy="0 0 0"/>
+      <geometry><box size="0.065 0.022 0.020"/></geometry>
+      <material name="motor_yellow"/>
+    </visual>
+    <!-- Visual: 4 Brass Standoff Pillars -->
+    <visual>
+      <origin xyz="0.075 0.060 ${lower_deck_z_pos + standoff_h/2}" rpy="0 0 0"/>
+      <geometry><cylinder radius="${standoff_r}" length="${standoff_h}"/></geometry>
+      <material name="brass_gold"/>
+    </visual>
+    <visual>
+      <origin xyz="0.075 -0.060 ${lower_deck_z_pos + standoff_h/2}" rpy="0 0 0"/>
+      <geometry><cylinder radius="${standoff_r}" length="${standoff_h}"/></geometry>
+      <material name="brass_gold"/>
+    </visual>
+    <visual>
+      <origin xyz="-0.075 0.060 ${lower_deck_z_pos + standoff_h/2}" rpy="0 0 0"/>
+      <geometry><cylinder radius="${standoff_r}" length="${standoff_h}"/></geometry>
+      <material name="brass_gold"/>
+    </visual>
+    <visual>
+      <origin xyz="-0.075 -0.060 ${lower_deck_z_pos + standoff_h/2}" rpy="0 0 0"/>
+      <geometry><cylinder radius="${standoff_r}" length="${standoff_h}"/></geometry>
+      <material name="brass_gold"/>
+    </visual>
+    <!-- Visual: Upper Chassis White Deck Plate -->
+    <visual>
+      <origin xyz="0 0 ${upper_deck_z_pos}" rpy="0 0 0"/>
+      <geometry><box size="${upper_deck_x} ${upper_deck_y} ${upper_deck_z}"/></geometry>
+      <material name="deck_white"/>
+    </visual>
+    <collision>
+      <origin xyz="0 0 ${upper_deck_z_pos}" rpy="0 0 0"/>
+      <geometry><box size="${upper_deck_x} ${upper_deck_y} ${upper_deck_z}"/></geometry>
+    </collision>
+    <!-- Visual: Battery Gauge Display on Side -->
+    <visual>
+      <origin xyz="0.020 0.072 ${lower_deck_z_pos + 0.005}" rpy="0 0 0"/>
+      <geometry><box size="0.045 0.010 0.020"/></geometry>
+      <material name="accent_blue"/>
+    </visual>
+    <xacro:box_inertia m="${lower_deck_mass + upper_deck_mass}" x="${lower_deck_x}" y="${lower_deck_y}" z="${upper_deck_z_pos}"/>
   </link>
   <joint name="base_footprint_joint" type="fixed">
@@ -101,32 +196,19 @@
   </joint>
   <!-- ============================================================
-       body_link : upper enclosure (visual / collision for nav height)
-       ============================================================ -->
-  <link name="body_link">
-    <visual>
-      <origin xyz="0 0 ${axle_height + base_z + 0.22}" rpy="0 0 0"/>
-      <geometry><box size="0.34 0.28 0.44"/></geometry>
-      <material name="body_white"/>
-    </visual>
-    <collision>
-      <origin xyz="0 0 ${axle_height + base_z + 0.22}" rpy="0 0 0"/>
-      <geometry><box size="0.34 0.28 0.44"/></geometry>
-    </collision>
-    <xacro:box_inertia m="4.0" x="0.34" y="0.28" z="0.44"/>
-  </link>
-  <joint name="body_joint" type="fixed">
-    <parent link="base_link"/>
-    <child  link="body_link"/>
-    <origin xyz="0 0 0" rpy="0 0 0"/>
-  </joint>
-  <!-- ============================================================
-       Drive wheels
-       ============================================================ -->
-  <xacro:macro name="drive_wheel" params="prefix side_y">
+       2. 4WD DRIVE WHEELS (Skid-Steer / 4-Wheel Drive)
+       ============================================================ -->
+  <xacro:macro name="drive_wheel" params="prefix pos_x side_y">
     <link name="${prefix}_wheel_link">
+      <!-- Rubber Tire Tread (Black) -->
       <visual>
         <origin xyz="0 0 0" rpy="${PI/2} 0 0"/>
         <geometry><cylinder radius="${wheel_radius}" length="${wheel_width}"/></geometry>
-        <material name="dark"/>
+        <material name="rubber_black"/>
+      </visual>
+      <!-- Yellow Rim Center -->
+      <visual>
+        <origin xyz="0 0 0" rpy="${PI/2} 0 0"/>
+        <geometry><cylinder radius="${wheel_radius * 0.78}" length="${wheel_width + 0.001}"/></geometry>
+        <material name="rim_yellow"/>
       </visual>
       <collision>
@@ -139,24 +221,25 @@
       <parent link="base_link"/>
       <child  link="${prefix}_wheel_link"/>
-      <origin xyz="0 ${side_y} ${axle_height}" rpy="0 0 0"/>
+      <origin xyz="${pos_x} ${side_y} ${axle_height}" rpy="0 0 0"/>
       <axis xyz="0 1 0"/>
     </joint>
   </xacro:macro>
-  <xacro:drive_wheel prefix="left"  side_y="${ wheel_separation/2}"/>
-  <xacro:drive_wheel prefix="right" side_y="${-wheel_separation/2}"/>
-  <!-- ============================================================
-       Rear caster (passive)
-       ============================================================ -->
+  <!-- 4 Independent Drive Wheels (Skid-Steer) -->
+  <xacro:drive_wheel prefix="front_left"  pos_x="${ wheelbase/2}" side_y="${ wheel_separation/2}"/>
+  <xacro:drive_wheel prefix="front_right" pos_x="${ wheelbase/2}" side_y="${-wheel_separation/2}"/>
+  <xacro:drive_wheel prefix="rear_left"   pos_x="${-wheelbase/2}" side_y="${ wheel_separation/2}"/>
+  <xacro:drive_wheel prefix="rear_right"  pos_x="${-wheelbase/2}" side_y="${-wheel_separation/2}"/>
+  <!-- Passive Caster Wheel Link (Virtual / Backwards Compatibility) -->
   <link name="caster_wheel_link">
     <visual>
-      <geometry><sphere radius="${caster_radius}"/></geometry>
-      <material name="dark"/>
-    </visual>
-    <collision>
-      <geometry><sphere radius="${caster_radius}"/></geometry>
+      <geometry><sphere radius="0.005"/></geometry>
+      <material name="rubber_black"/>
+    </visual>
+    <collision>
+      <geometry><sphere radius="0.005"/></geometry>
     </collision>
     <inertial>
-      <mass value="0.1"/>
-      <inertia ixx="0.00002" ixy="0" ixz="0" iyy="0.00002" iyz="0" izz="0.00002"/>
+      <mass value="0.01"/>
+      <inertia ixx="0.000001" ixy="0" ixz="0" iyy="0.000001" iyz="0" izz="0.000001"/>
     </inertial>
   </link>
@@ -164,19 +247,34 @@
     <parent link="base_link"/>
     <child  link="caster_wheel_link"/>
-    <origin xyz="${caster_x} 0 ${caster_radius}" rpy="0 0 0"/>
-  </joint>
-  <!-- ============================================================
-       2D LiDAR  ->  frame name MUST match the driver's frame_id
-       and rf2o's laser frame:  laser_frame
+    <origin xyz="-0.080 0 0.005" rpy="0 0 0"/>
+  </joint>
+  <!-- ============================================================
+       3. 2D LIDAR (Slamtec RPLiDAR A1)
+          TF frame: laser_frame (must match sllidar_node & rf2o)
        ============================================================ -->
   <link name="laser_frame">
-    <visual>
-      <geometry><cylinder radius="0.045" length="0.04"/></geometry>
+    <!-- Elevated Black Riser Mount Plate -->
+    <visual>
+      <origin xyz="0 0 -0.040" rpy="0 0 0"/>
+      <geometry><box size="${lidar_riser_x} ${lidar_riser_y} ${lidar_riser_z}"/></geometry>
+      <material name="chassis_black"/>
+    </visual>
+    <!-- RPLiDAR A1 Rotating Turret -->
+    <visual>
+      <origin xyz="0 0 0" rpy="0 0 0"/>
+      <geometry><cylinder radius="0.035" length="0.040"/></geometry>
       <material name="sensor_black"/>
     </visual>
-    <collision>
-      <geometry><cylinder radius="0.045" length="0.04"/></geometry>
-    </collision>
-    <xacro:cylinder_inertia m="0.2" r="0.045" l="0.04"/>
+    <!-- Secondary Belt Drive Motor on Side -->
+    <visual>
+      <origin xyz="-0.032 0 -0.010" rpy="0 0 0"/>
+      <geometry><cylinder radius="0.012" length="0.025"/></geometry>
+      <material name="sensor_black"/>
+    </visual>
+    <collision>
+      <origin xyz="0 0 0" rpy="0 0 0"/>
+      <geometry><cylinder radius="0.038" length="0.045"/></geometry>
+    </collision>
+    <xacro:cylinder_inertia m="${lidar_mass}" r="0.038" l="0.045"/>
   </link>
   <joint name="laser_joint" type="fixed">
@@ -185,14 +283,47 @@
     <origin xyz="${lidar_x} ${lidar_y} ${lidar_z}" rpy="0 0 ${lidar_yaw}"/>
   </joint>
-  <!-- ============================================================
-       Camera : body frame + REP-103 optical frame
-       (optical frame: z forward, x right, y down)
+  <!-- Optional lidar_link alias for packages expecting lidar_link frame -->
+  <link name="lidar_link"/>
+  <joint name="lidar_link_alias_joint" type="fixed">
+    <parent link="laser_frame"/>
+    <child  link="lidar_link"/>
+    <origin xyz="0 0 0" rpy="0 0 0"/>
+  </joint>
+  <!-- ============================================================
+       4. UPPER COMPANION BODY / HEAD SHELL (3D Printed Enclosure)
+       ============================================================ -->
+  <link name="body_link">
+    <!-- Main Upper Body Shell (White) -->
+    <visual>
+      <origin xyz="0 0 0" rpy="0 0 0"/>
+      <geometry><box size="${head_length} ${head_width} ${head_height}"/></geometry>
+      <material name="shell_white"/>
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